File: WemosMosfet.kicad_pcb (KiCad board)
At the start: 2 copper layers, 35.6 x 27 mm, 26 parts, among them J1 MIST, J2 ADC_1, J3 KEY_2, J4 KEY_1, Q1 BSS84, Q2 BSS84, Q3 BSS138, Q5 BSS138, Q7 BSS138, U1 WeMos_D1_mini

Commit message: Fixed some design flaws, first version didn't work.
Parts:
- removed R8: 18K, Resistor_SMD:R_0805_2012Metric_Pad1.20x1.40mm_HandSolder
- added R6: 10K, Resistor_SMD:R_0805_2012Metric_Pad1.20x1.40mm_HandSolder, F.Cu at (28.8, 23.4)
Connections:
- Q3 pad 2: Net-(Q3-S) -> GND
- Q5 pad 2: Net-(Q5-S) -> GND
- Q5 pad 3: Net-(Q1-G) -> Net-(Q5-D)
- Q7 pad 2: Net-(Q7-S) -> GND
- Q7 pad 3: Net-(Q2-G) -> Net-(Q7-D)
- R1 pad 1: GND -> Net-(Q5-D)
- R1 pad 2: Net-(Q5-S) -> Net-(Q1-G)
- R2 pad 1: GND -> Net-(Q7-D)
- R2 pad 2: Net-(Q7-S) -> Net-(Q2-G)
Routing:
- net Net-(Q5-S): track 4.73 -> 0.00 mm
- net Net-(Q3-S): track 4.43 -> 0.00 mm
- net Net-(Q7-S): track 4.21 -> 0.00 mm
- net +3.3V: track 6.87 -> 9.92 mm
- net Net-(Q7-D): track 0.00 -> 2.92 mm
- net Net-(Q5-D): track 0.00 -> 2.92 mm
- net Net-(Q1-G): track 6.94 -> 7.72 mm
- net Net-(Q2-G): track 6.94 -> 7.72 mm
- net Net-(Q3-D): track 27.9 -> 28.7 mm
